File: board/icemot/icemot_v1/icemotv1.sch (EAGLE design)
At the start: 20 parts, among them U1 ICE40HX4K, U2 EFM32WG332FXXX-QFP64, Y1 48MHz

Commit message: starting ICE schematic
Connections:
- new net +1V2: U1F.VCC@111, U1F.VCC@27, U1F.VCC@40, U1F.VCC@92
- net GND: now also U1F.GND@103, U1F.GND@13, U1F.GND@132, U1F.GND@14, U1F.GND@140, U1F.GND@5, U1F.GND@59, U1F.GND@69, U1F.GND@86
Changed lines of the file:
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@@
 <part name="SUPPLY20" library="supply2" deviceset="GND" device=""/>
 <part name="SUPPLY21" library="supply2" deviceset="GND" device=""/>
+<part name="U$2" library="symbols" deviceset="+1V2" device=""/>
+<part name="SUPPLY22" library="supply2" deviceset="GND" device=""/>
 </parts>
 <sheets>
@@
 <instance part="U1" gate="E" x="182.88" y="134.62"/>
 <instance part="U1" gate="F" x="182.88" y="86.36"/>
+<instance part="U$2" gate="G$1" x="213.36" y="78.74"/>
+<instance part="SUPPLY22" gate="GND" x="152.4" y="78.74" smashed="yes">
+<attribute name="VALUE" x="150.495" y="75.565" size="1.778" layer="96" display="off"/>
+</instance>
 </instances>
 <busses>
 </busses>
 <nets>
+<net name="+1V2" class="0">
+<segment>
+<pinref part="U1" gate="F" pin="VCC@111"/>
+<pinref part="U$2" gate="G$1" pin="+1V2"/>
+<wire x1="205.74" y1="66.04" x2="213.36" y2="66.04" width="0.1524" layer="91"/>
+<wire x1="213.36" y1="66.04" x2="213.36" y2="68.58" width="0.1524" layer="91"/>
+<pinref part="U1" gate="F" pin="VCC@92"/>
+<wire x1="213.36" y1="68.58" x2="213.36" y2="71.12" width="0.1524" layer="91"/>
+<wire x1="213.36" y1="71.12" x2="213.36" y2="73.66" width="0.1524" layer="91"/>
+<wire x1="213.36" y1="73.66" x2="213.36" y2="76.2" width="0.1524" layer="91"/>
+<wire x1="205.74" y1="68.58" x2="213.36" y2="68.58" width="0.1524" layer="91"/>
+<junction x="213.36" y="68.58"/>
+<pinref part="U1" gate="F" pin="VCC@40"/>
+<wire x1="205.74" y1="71.12" x2="213.36" y2="71.12" width="0.1524" layer="91"/>
+<junction x="213.36" y="71.12"/>
+<pinref part="U1" gate="F" pin="VCC@27"/>
+<wire x1="205.74" y1="73.66" x2="213.36" y2="73.66" width="0.1524" layer="91"/>
+<junction x="213.36" y="73.66"/>
+</segment>
+</net>
+<net name="GND" class="0">
+<segment>
+<pinref part="U1" gate="F" pin="GND@5"/>
+<pinref part="SUPPLY22" gate="GND" pin="GND"/>
+<wire x1="160.02" y1="104.14" x2="152.4" y2="104.14" width="0.1524" layer="91"/>
+<wire x1="152.4" y1="104.14" x2="152.4" y2="101.6" width="0.1524" layer="91"/>
+<pinref part="U1" gate="F" pin="GND@140"/>
+<wire x1="152.4" y1="101.6" x2="152.4" y2="99.06" width="0.1524" layer="91"/>
+<wire x1="152.4" y1="99.06" x2="152.4" y2="96.52" width="0.1524" layer="91"/>
+<wire x1="152.4" y1="96.52" x2="152.4" y2="93.98" width="0.1524" layer="91"/>
+<wire x1="152.4" y1="93.98" x2="152.4" y2="91.44" width="0.1524" layer="91"/>
+<wire x1="152.4" y1="91.44" x2="152.4" y2="88.9" width="0.1524" layer="91"/>
+<wire x1="152.4" y1="88.9" x2="152.4" y2="86.36" width="0.1524" layer="91"/>
+<wire x1="152.4" y1="86.36" x2="152.4" y2="83.82" width="0.1524" layer="91"/>
+<wire x1="152.4" y1="83.82" x2="152.4" y2="81.28" width="0.1524" layer="91"/>
+<wire x1="160.02" y1="83.82" x2="152.4" y2="83.82" width="0.1524" layer="91"/>
+<junction x="152.4" y="83.82"/>
+<pinref part="U1" gate="F" pin="GND@132"/>
+<wire x1="160.02" y1="86.36" x2="152.4" y2="86.36" width="0.1524" layer="91"/>
+<junction x="152.4" y="86.36"/>
+<pinref part="U1" gate="F" pin="GND@103"/>
+<wire x1="160.02" y1="88.9" x2="152.4" y2="88.9" width="0.1524" layer="91"/>
+<junction x="152.4" y="88.9"/>
+<pinref part="U1" gate="F" pin="GND@86"/>
+<wire x1="160.02" y1="91.44" x2="152.4" y2="91.44" width="0.1524" layer="91"/>
+<junction x="152.4" y="91.44"/>
+<pinref part="U1" gate="F" pin="GND@69"/>
+<wire x1="160.02" y1="93.98" x2="152.4" y2="93.98" width="0.1524" layer="91"/>
+<junction x="152.4" y="93.98"/>
+<pinref part="U1" gate="F" pin="GND@59"/>
+<wire x1="160.02" y1="96.52" x2="152.4" y2="96.52" width="0.1524" layer="91"/>
+<junction x="152.4" y="96.52"/>
+<pinref part="U1" gate="F" pin="GND@14"/>
+<wire x1="160.02" y1="99.06" x2="152.4" y2="99.06" width="0.1524" layer="91"/>
+<junction x="152.4" y="99.06"/>
+<pinref part="U1" gate="F" pin="GND@13"/>
+<wire x1="160.02" y1="101.6" x2="152.4" y2="101.6" width="0.1524" layer="91"/>
+<junction x="152.4" y="101.6"/>
+</segment>
+</net>
 </nets>
 </sheet>

Commit message: need to add interface to motor
Parts:
- added C15, C16, C19, C20, C21, C22, C23, C24, C25, C26, C27, C28, C29, C30, C31, C39, C42, C43, C44, C45: 100n, standard_passive:CAP_0603
- added C17: 10uF, standard_passive:CAP_0805
- added C18: 10u, standard_passive:CAP_0805
- added C32, C41: 10n, standard_passive:CAP_0603
- added C33, C35, C36: 0.1u, standard_passive:CAP_0603
- added C34: 0.47u, standard_passive:CAP_0603
- added C37, C38: (no value), rcl:CPOL-EUE5-5
- added C40: 1u, standard_passive:CAP_0603
- added D1: (no value), diode:DIODE-SOD123
- added JP1, JP2, JP3, JP4: (no value), pinhead:PINHD-1X2
- added R10: 1M, standard_passive:RES_0603
- added R11, R12, R13, R14: TBD, standard_passive:RES_0603
- added R3, R4: 100, standard_passive:RES_0603
- added R5, R6, R7: 10k, standard_passive:RES_0603
- added R8, R9: 0.1, standard_passive:RES_1206
- added U$4: DRV8825PWP, motor_drivers:DRV8825PWP
- added U3: MAX5723/4/5, dac:MAX5723/4/5
- added U4: TLV4379, opamp:TLV4379
- added X1: MSTBV4, con-phoenix-508:MSTBV4
Connections:
- new net CDONE: R6.1, U1C.CDONE
- new net CONF_CS: R5.2, U1E.PIOS_03/SPI_SS_B, U2.PE13@62
- new net CONF_MISO: U1E.PIOS_02/SPI_SO, U2.PE11@60, U3.DOUT@12
- new net CONF_MOSI: U1E.PIOS_01/SPI_SI, U2.PE10@59, U3.DIN@13
- new net CONF_SCK: U1E.PIOS_00/SPI_SCK, U2.PE12@61, U3.SCK@14
- new net CRESET: R7.1, U1C.CRESET_B
- new net DAC_CS: U2.PE14@63, U3.CSB@15
- new net MOT1_REF: U3.OUT0@2
- new net N$10: C16.1, C18.1, R4.2, U1F.PLLVCC@54
- new net N$11: C15.1, C17.1, R3.2, U1F.PLLVCC@126
- new net N$12: C15.2, C17.2, U1F.PLLGND@127
- new net N$13: C16.2, C18.2, U1F.PLLGND@53
- new net N$14: D1.C, U1F.VPP_2V5
- new net N$15: U2.PE15@64
- new net N$16: R9.2, U$4.ISENA
- new net N$17: R8.2, U$4.ISENB
- new net N$18: C32.1, U$4.CP1
- new net N$19: C32.2, U$4.CP2
- new net N$20: C33.1, R10.1, U$4.VCP
- new net N$21: U$4.AVREF, U$4.BVREF
- new net N$22: U$4.RESET, U$4.SLEEP
- new net N$23: U$4.FAULT
- new net N$24: U$4.DECAY
- new net N$25: U$4.DIR
- new net N$26: U$4.STEP
- new net N$27: U$4.ENBL
- new net N$29: U$4.AOUT1, X1-4.1
- new net N$30: U$4.AOUT2, X1-3.1
- new net N$31: U$4.BOUT2, X1-2.1
- new net N$32: U$4.BOUT1, X1-1.1
- new net N$34: U3.OUT1@3
- new net N$35: U3.OUT2@4
- new net N$36: U3.OUT3@5
- new net N$37: U3.OUT4@6
- new net N$38: U3.OUT5@7
- new net N$39: U3.OUT6@8
- new net N$40: U3.OUT7@9
- new net T1_AMP: U2.PD3@31, U4.A_N@2, U4.OUT_A@1
- new net T1_IN: C42.1, JP1.1, R11.2, U4.A_P@3
- new net T2_AMP: U2.PD4@32, U4.B_N@6, U4.OUT_B@7
- new net T2_IN: C43.1, JP2.1, R12.2, U4.B_P@5
- new net T3_AMP: U2.PD5@33, U4.C_N@9, U4.OUT_C@8
- new net T3_IN: C44.1, JP3.1, R13.2, U4.C_P@10
- new net T4_AMP: U2.PD6@34, U4.D_N@13, U4.OUT_D@14
- new net T4_IN: C45.1, JP4.1, R14.2, U4.D_P@12
- net +1V2: now also C19.1, C20.1, C21.1, C22.1, C33.2, C35.1, C36.1, C37.+, C38.+, R10.2, R3.1, R4.1, U$4.VMA, U$4.VMB
- net +3V3: now also C23.1, C24.1, C25.1, C26.1, C27.1, C28.1, C29.1, C30.1, C31.1, C34.2, C39.1, C40.1, C41.1, D1.A, JP1.2, JP2.2, JP3.2, JP4.2, R6.2, R7.2, U$4.MODE0, U$4.MODE1, U$4.MODE2, U$4.V3P3OUT, U1C.VCCIO2@46, U1C.VCCIO2@57, U1E.SPI_VCC, U3.NCLR@17, U3.NLDAC@18, U3.VDD@10, U3.VDDIO@11, U4.V+@4
- net GND: now also C19.2, C20.2, C21.2, C22.2, C23.2, C24.2, C25.2, C26.2, C27.2, C28.2, C29.2, C30.2, C31.2, C34.1, C35.2, C36.2, C37.-, C38.-, C39.2, C40.2, C41.2, C42.2, C43.2, C44.2, C45.2, R11.1, R12.1, R13.1, R14.1, R5.1, R8.1, R9.1, U$4.GND_0, U$4.GND_1, U$4.GND_PAD, U3.GND@19, U3.MNZ@20, U4.V-@11
Other:
- note added: "100VDC Ceramic cap !"
- note added: "WHY ?!"
- note added: "iCE40sysCLOCKPLLDesignandUsageGuide p.18"

Commit message: added oscillator, clock to be routed on GBin
Parts:
- added C46: 0.47u, standard_passive:CAP_0603
- added C47, C48: 0.1u, standard_passive:CAP_0603
- added U$6: 3.2X2.5X2.0-TCXO, oscillators:3.2X2.5X2.0-TCXO
Connections:
- removed net MOT1_REF: U3.OUT0@2
- removed net N$21: U$4.AVREF, U$4.BVREF
- new net +40V: C33.2, C35.1, C36.1, C37.+, C38.+, R10.2, U$4.VMA, U$4.VMB
- new net +40V1: C47.1, C48.1
- new net MOT1_VREF: C46.1, U$4.AVREF, U$4.BVREF, U3.OUT0@2
- net +1V2: no longer C33.2, C35.1, C36.1, C37.+, C38.+, R10.2, U$4.VMA, U$4.VMB
- net GND: now also C46.2, C47.2, C48.2
- net N$29: now also X1-1.1; no longer X1-4.1
- net N$30: now also X1-2.1; no longer X1-3.1
- net N$31: now also X1-3.1; no longer X1-2.1
- net N$32: now also X1-4.1; no longer X1-1.1
Other:
- moved on the sheet: X1-1, X1-2, X1-3, X1-4

Commit message: added res on decay
Parts:
- added C49: 100n, standard_passive:CAP_0603
- added R15: 0, standard_passive:RES_0603
- added R16: 10k, standard_passive:RES_0603
Connections:
- removed net N$22: U$4.RESET, U$4.SLEEP
- removed net N$23: U$4.FAULT
- removed net N$25: U$4.DIR
- removed net N$26: U$4.STEP
- removed net N$27: U$4.ENBL
- new net MOT1_DIR: U$4.DIR, U1C.PIO2_14
- new net MOT1_EN: U$4.ENBL, U1C.PIO2_15
- new net MOT1_FAULT: R16.1, U$4.FAULT, U1C.PIO2_16
- new net MOT1_RST: U$4.RESET, U$4.SLEEP, U1C.PIO2_12
- new net MOT1_STEP: U$4.STEP, U1C.PIO2_13
- new net N$21: U$6.OUT, U1D.GBIN6/PIO3_00/DP08A
- net +3V3: now also C49.1, R15.1, R16.2, U$6.VDD
- net GND: now also C49.2, U$6.GND
- net N$24: now also R15.2
Changed lines of the file:
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@@
 <setting verticaltext="up"/>
 </settings>
-<grid distance="0.1" unitdist="inch" unit="inch" style="lines" multiple="1" display="no" altdistance="0.01" altunitdist="inch" altunit="inch"/>
+<grid distance="0.1" unitdist="inch" unit="inch" style="lines" multiple="1" display="yes" altdistance="0.01" altunitdist="inch" altunit="inch"/>
 <layers>
 <layer number="1" name="Top" color="4" fill="1" visible="no" active="no"/>
@@
 <part name="SUPPLY55" library="supply2" deviceset="GND" device=""/>
 <part name="U$6" library="oscillators" deviceset="3.2X2.5X2.0-TCXO" device=""/>
+<part name="C49" library="standard_passive" deviceset="CAP_0603" device="" value="100n"/>
+<part name="SUPPLY56" library="supply2" deviceset="GND" device=""/>
+<part name="SUPPLY57" library="supply2" deviceset="GND" device=""/>
+<part name="+3V25" library="supply1" deviceset="+3V3" device=""/>
+<part name="R15" library="standard_passive" deviceset="RES_0603" device="" value="0"/>
+<part name="R16" library="standard_passive" deviceset="RES_0603" device="" value="10k"/>
+<part name="+3V26" library="supply1" deviceset="+3V3" device=""/>
 </parts>
 <sheets>
@@
 </instance>
 <instance part="U$6" gate="G$1" x="58.42" y="33.02"/>
+<instance part="C49" gate="G$1" x="33.02" y="33.02"/>
+<instance part="SUPPLY56" gate="GND" x="43.18" y="22.86" smashed="yes">
+<attribute name="VALUE" x="41.275" y="19.685" size="1.778" layer="96" display="off"/>
+</instance>
+<instance part="SUPPLY57" gate="GND" x="33.02" y="22.86" smashed="yes">
+<attribute name="VALUE" x="31.115" y="19.685" size="1.778" layer="96" display="off"/>
+</instance>
+<instance part="+3V25" gate="G$1" x="33.02" y="48.26"/>
 </instances>
 <busses>
@@
 <wire x1="81.28" y1="88.9" x2="81.28" y2="86.36" width="0.1524" layer="91"/>
 </segment>
+<segment>
+<pinref part="U$6" gate="G$1" pin="GND"/>
+<wire x1="45.72" y1="27.94" x2="43.18" y2="27.94" width="0.1524" layer="91"/>
+<pinref part="SUPPLY56" gate="GND" pin="GND"/>
+<wire x1="43.18" y1="27.94" x2="43.18" y2="25.4" width="0.1524" layer="91"/>
+</segment>
+<segment>
+<pinref part="C49" gate="G$1" pin="2"/>
+<pinref part="SUPPLY57" gate="GND" pin="GND"/>
+<wire x1="33.02" y1="27.94" x2="33.02" y2="25.4" width="0.1524" layer="91"/>
+</segment>
 </net>
 <net name="N$10" class="0">
@@
 <wire x1="81.28" y1="99.06" x2="81.28" y2="96.52" width="0.1524" layer="91"/>
 </segment>
+<segment>
+<pinref part="+3V25" gate="G$1" pin="+3V3"/>
+<pinref part="C49" gate="G$1" pin="1"/>
+<wire x1="33.02" y1="45.72" x2="33.02" y2="38.1" width="0.1524" layer="91"/>
+<pinref part="U$6" gate="G$1" pin="VDD"/>
+<wire x1="33.02" y1="38.1" x2="33.02" y2="35.56" width="0.1524" layer="91"/>
+<wire x1="45.72" y1="38.1" x2="33.02" y2="38.1" width="0.1524" layer="91"/>
+<junction x="33.02" y="38.1"/>
+</segment>
 </net>
 <net name="CONF_CS" class="0">
@@
 <junction x="269.24" y="170.18"/>
 <label x="256.54" y="170.18" size="1.778" layer="95"/>
+</segment>
+</net>
+<net name="N$21" class="0">
+<segment>
+<pinref part="U$6" gate="G$1" pin="OUT"/>
+<pinref part="U1" gate="D" pin="GBIN6/PIO3_00/DP08A"/>
+<wire x1="71.12" y1="33.02" x2="96.52" y2="33.02" width="0.1524" layer="91"/>
+</segment>
+</net>
+<net name="MOT1_FAULT" class="0">
+<segment>
+<pinref part="U1" gate="C" pin="PIO2_16"/>
+<wire x1="345.44" y1="162.56" x2="363.22" y2="162.56" width="0.1524" layer="91"/>
+<label x="350.52" y="162.56" size="1.778" layer="95"/>
+</segment>
+</net>
+<net name="MOT1_EN" class="0">
+<segment>
+<pinref part="U1" gate="C" pin="PIO2_15"/>
+<wire x1="345.44" y1="165.1" x2="363.22" y2="165.1" width="0.1524" layer="91"/>
+<label x="350.52" y="165.1" size="1.778" layer="95"/>
+</segment>
+</net>
+<net name="MOT1_DIR" class="0">
+<segment>
+<pinref part="U1" gate="C" pin="PIO2_14"/>
+<wire x1="345.44" y1="167.64" x2="363.22" y2="167.64" width="0.1524" layer="91"/>
+<label x="350.52" y="167.64" size="1.778" layer="95"/>
+</segment>
+</net>
+<net name="MOT1_STEP" class="0">
+<segment>
+<pinref part="U1" gate="C" pin="PIO2_13"/>
+<wire x1="345.44" y1="170.18" x2="363.22" y2="170.18" width="0.1524" layer="91"/>
+<label x="350.52" y="170.18" size="1.778" layer="95"/>
+</segment>
+</net>
+<net name="MOT1_RST" class="0">
+<segment>
+<pinref part="U1" gate="C" pin="PIO2_12"/>
+<wire x1="345.44" y1="172.72" x2="363.22" y2="172.72" width="0.1524" layer="91"/>
+<label x="350.52" y="172.72" size="1.778" layer="95"/>
 </segment>
 </net>
@@
 <attribute name="VALUE" x="149.225" y="167.005" size="1.778" layer="96" rot="R270" display="off"/>
 </instance>
-<instance part="+3V15" gate="G$1" x="152.4" y="132.08" rot="R90"/>
+<instance part="+3V15" gate="G$1" x="137.16" y="132.08" smashed="yes" rot="R90">
+<attribute name="VALUE" x="142.24" y="137.16" size="1.778" layer="96" rot="R180"/>
+</instance>
 <instance part="C35" gate="G$1" x="248.92" y="132.08" smashed="yes" rot="R90">
 <attribute name="NAME" x="248.412" y="134.239" size="1.778" layer="95" rot="R180"/>
@@
 <attribute name="VALUE" x="267.335" y="160.655" size="1.778" layer="96" rot="R90" display="off"/>
 </instance>
+<instance part="R15" gate="G$1" x="154.94" y="137.16" smashed="yes">
+<attribute name="NAME" x="148.59" y="133.5786" size="1.778" layer="95"/>
+<attribute name="VALUE" x="158.75" y="133.858" size="1.778" layer="96"/>
+</instance>
+<instance part="R16" gate="G$1" x="116.84" y="124.46" smashed="yes" rot="R90">
+<attribute name="NAME" x="120.4214" y="118.11" size="1.778" layer="95" rot="R90"/>
+<attribute name="VALUE" x="120.142" y="128.27" size="1.778" layer="96" rot="R90"/>
+</instance>
+<instance part="+3V26" gate="G$1" x="116.84" y="134.62"/>
 </instances>
 <busses>
@@
 <junction x="165.1" y="132.08"/>
 <pinref part="+3V15" gate="G$1" pin="+3V3"/>
-<wire x1="154.94" y1="132.08" x2="165.1" y2="132.08" width="0.1524" layer="91"/>
+<wire x1="139.7" y1="132.08" x2="144.78" y2="132.08" width="0.1524" layer="91"/>
+<pinref part="R15" gate="G$1" pin="1"/>
+<wire x1="144.78" y1="132.08" x2="165.1" y2="132.08" width="0.1524" layer="91"/>
+<wire x1="149.86" y1="137.16" x2="144.78" y2="137.16" width="0.1524" layer="91"/>
+<wire x1="144.78" y1="137.16" x2="144.78" y2="132.08" width="0.1524" layer="91"/>
+<junction x="144.78" y="132.08"/>
+</segment>
+<segment>
+<pinref part="+3V26" gate="G$1" pin="+3V3"/>
+<pinref part="R16" gate="G$1" pin="2"/>
+<wire x1="116.84" y1="132.08" x2="116.84" y2="129.54" width="0.1524" layer="91"/>
 </segment>
 </net>
@@
 </segment>
 </net>
-<net name="N$22" class="0">
+<net name="MOT1_RST" class="0">
 <segment>
 <pinref part="U$4" gate="G$1" pin="RESET"/>
 <wire x1="172.72" y1="127" x2="160.02" y2="127" width="0.1524" layer="91"/>
 <pinref part="U$4" gate="G$1" pin="SLEEP"/>
-<wire x1="160.02" y1="127" x2="137.16" y2="127" width="0.1524" layer="91"/>
+<wire x1="160.02" y1="127" x2="121.92" y2="127" width="0.1524" layer="91"/>
 <wire x1="172.72" y1="124.46" x2="160.02" y2="124.46" width="0.1524" layer="91"/>
 <wire x1="160.02" y1="124.46" x2="160.02" y2="127" width="0.1524" layer="91"/>
 <junction x="160.02" y="127"/>
-</segment>
-</net>
-<net name="N$23" class="0">
+<label x="124.46" y="127" size="1.778" layer="95"/>
+</segment>
+</net>
+<net name="MOT1_FAULT" class="0">
 <segment>
 <pinref part="U$4" gate="G$1" pin="FAULT"/>
-<wire x1="172.72" y1="116.84" x2="137.16" y2="116.84" width="0.1524" layer="91"/>
-</segment>
-</net>
-<net name="N$24" class="0">
-<segment>
-<pinref part="U$4" gate="G$1" pin="DECAY"/>
-<wire x1="172.72" y1="137.16" x2="137.16" y2="137.16" width="0.1524" layer="91"/>
-</segment>
-</net>
-<net name="N$25" class="0">
+<wire x1="172.72" y1="116.84" x2="116.84" y2="116.84" width="0.1524" layer="91"/>
+<pinref part="R16" gate="G$1" pin="1"/>
+<wire x1="116.84" y1="116.84" x2="116.84" y2="119.38" width="0.1524" layer="91"/>
+<label x="121.92" y="116.84" size="1.778" layer="95"/>
+</segment>
+</net>
+<net name="MOT1_DIR" class="0">
 <segment>
 <pinref part="U$4" gate="G$1" pin="DIR"/>
 <wire x1="172.72" y1="139.7" x2="137.16" y2="139.7" width="0.1524" layer="91"/>
-</segment>
-</net>
-<net name="N$26" class="0">
+<label x="139.7" y="139.7" size="1.778" layer="95"/>
+</segment>
+</net>
+<net name="MOT1_STEP" class="0">
 <segment>
 <pinref part="U$4" gate="G$1" pin="STEP"/>
 <wire x1="172.72" y1="142.24" x2="137.16" y2="142.24" width="0.1524" layer="91"/>
-</segment>
-</net>
-<net name="N$27" class="0">
+<label x="139.7" y="142.24" size="1.778" layer="95"/>
+</segment>
+</net>
+<net name="MOT1_EN" class="0">
 <segment>
 <pinref part="U$4" gate="G$1" pin="ENBL"/>
 <wire x1="172.72" y1="144.78" x2="137.16" y2="144.78" width="0.1524" layer="91"/>
+<label x="139.7" y="144.78" size="1.778" layer="95"/>
 </segment>
 </net>
@@
 </segment>
 </net>
+<net name="N$24" class="0">
+<segment>
+<pinref part="R15" gate="G$1" pin="2"/>
+<pinref part="U$4" gate="G$1" pin="DECAY"/>
+<wire x1="160.02" y1="137.16" x2="172.72" y2="137.16" width="0.1524" layer="91"/>
+</segment>
+</net>

Commit message: remove ICE40 and EFM32, add a S6 LX9
Parts:
- removed C10, C15, C16, C19, C20, C21, C22, C23, C24, C25, C26, C27, C28, C29, C3, C30, C31, C5, C6, C7, C8: 100n, standard_passive:CAP_0603
- removed C11: 4.7u, standard_passive:CAP_0805
- removed C12: 1u, standard_passive:CAP_0603
- removed C13, C14: 10p, standard_passive:CAP_0603
- removed C17: 10uF, standard_passive:CAP_0805
- removed C18, C2, C4, C9: 10u, standard_passive:CAP_0805
- removed D1: (no value), diode:DIODE-SOD123
- removed R1, R2: 15, standard_passive:RES_0603
- removed R3, R4: 100, standard_passive:RES_0603
- removed R5, R6, R7: 10k, standard_passive:RES_0603
- removed U$1: USB-SHIELD, usb-header:USB-SHIELD
- removed U2: EFM32WG332FXXX-QFP64, EFM32:EFM32WG332FXXX-QFP64
- removed Y1: 48MHz, xtals:CRYSTAL.3.2X2.5MM
- U1: value ICE40HX4K -> 6SLX9TQG144; device ICE40HX:ICE40HX4K -> xilinx:6SLX9TQG144
Connections:
- removed net +1V2: C19.1, C20.1, C21.1, C22.1, R3.1, R4.1, U1F.VCC@111, U1F.VCC@27, U1F.VCC@40, U1F.VCC@92
- removed net CDONE: R6.1, U1C.CDONE
- removed net CONF_CS: R5.2, U1E.PIOS_03/SPI_SS_B, U2.PE13@62
- removed net CRESET: R7.1, U1C.CRESET_B
- removed net N$1: C1.1, U2.DECOUPLE@40
- removed net N$10: C16.1, C18.1, R4.2, U1F.PLLVCC@54
- removed net N$11: C15.1, C17.1, R3.2, U1F.PLLVCC@126
- removed net N$12: C15.2, C17.2, U1F.PLLGND@127
- removed net N$13: C16.2, C18.2, U1F.PLLGND@53
- removed net N$14: D1.C, U1F.VPP_2V5
- removed net N$15: U2.PE15@64
- removed net N$2: R1.1, U2.PF10_USBDM@47
- removed net N$21: U$6.OUT, U1D.GBIN6/PIO3_00/DP08A
- removed net N$3: R1.2, U$1.D-
- removed net N$4: C11.1, U$1.VBUS, U2.USBVBUS@52, U2.USBVREGI@45
- removed net N$5: C12.2, U2.USBVREGO@46
- removed net N$6: R2.2, U$1.D+
- removed net N$7: R2.1, U2.PF11_USBDP@48
- removed net N$8: C13.1, U2.PB14_HFXTALN@25, Y1.2
- removed net N$9: C14.1, U2.PB13_HFXTALP@24, Y1.1
- net +3V3: now also C1.1; no longer C10.2, C2.1, C23.1, C24.1, C25.1, C26.1, C27.1, C28.1, C29.1, C3.1, C30.1, C31.1, C4.1, C5.1, C6.1, C7.1, C8.1, C9.1, D1.A, R6.2, R7.2, U1C.VCCIO2@46, U1C.VCCIO2@57, U1E.SPI_VCC, U2.AVDD@23, U2.AVDD@27, U2.IOVDD@26, U2.IOVDD@55, U2.IOVDD@7, U2.VDDREG@39
- net CONF_MISO: no longer U1E.PIOS_02/SPI_SO, U2.PE11@60
- net CONF_MOSI: no longer U1E.PIOS_01/SPI_SI, U2.PE10@59
- net CONF_SCK: no longer U1E.PIOS_00/SPI_SCK, U2.PE12@61
- net DAC_CS: no longer U2.PE14@63
- net GND: no longer C10.1, C11.2, C12.1, C13.2, C14.2, C19.2, C2.2, C20.2, C21.2, C22.2, C23.2, C24.2, C25.2, C26.2, C27.2, C28.2, C29.2, C3.2, C30.2, C31.2, C4.2, C5.2, C6.2, C7.2, C8.2, C9.2, R5.1, U$1.GND, U$1.GND@1, U$1.GND@2, U$1.GND@3, U$1.GND@4, U1F.GND@103, U1F.GND@13, U1F.GND@132, U1F.GND@14, U1F.GND@140, U1F.GND@5, U1F.GND@59, U1F.GND@69, U1F.GND@86, U2.VSS@22, U2.VSS@56, U2.VSS@8
- net MOT1_DIR: no longer U1C.PIO2_14
- net MOT1_EN: no longer U1C.PIO2_15
- net MOT1_FAULT: no longer U1C.PIO2_16
- net MOT1_RST: no longer U1C.PIO2_12
- net MOT1_STEP: no longer U1C.PIO2_13
- net T1_AMP: no longer U2.PD3@31
- net T2_AMP: no longer U2.PD4@32
- net T3_AMP: no longer U2.PD5@33
- net T4_AMP: no longer U2.PD6@34
Other:
- note removed: "WHY ?!"
- note removed: "iCE40sysCLOCKPLLDesignandUsageGuide p.18"
