File: board/icemot/icemot_v1/icemotv1.sch (EAGLE design)
At the start: 38 parts, among them U1 6SLX9TQG144, U3 MAX5723/4/5, U4 TLV4379, X1 MSTBV4

Commit message: added ADC DCDC and copied 5 drv8825
Parts:
- added C10, C12, C13, C17, C18, C20, C22, C23, C27, C28, C3, C5, C50, C52, C53, C57, C58, C6, C65, C66: 0.1u, standard_passive:CAP_0603
- added C11, C16, C21, C26, C4, C51, C56, C64: 0.47u, standard_passive:CAP_0603
- added C14, C15, C24, C25, C54, C55, C7, C8: (no value), rcl:CPOL-EUE5-5
- added C19, C2, C31, C9: 10n, standard_passive:CAP_0603
- added C29, C30, C59, C62, C63, C67, C68, C69, C70, C71, C73, C76, C79, C82: 4.7u, rcl:C-EUC0603
- added C60, C61, C72, C74, C75, C77, C78, C80, C81, C83, C84: 470n, rcl:C-EUC0603
- added C85, C86, C87, C88: (no value), rcl:CPOL-EUE5-10.5
- added D1: MBR360G, diode:SCHOTTKY-DIODEDO201T15
- added L1: 100UH, Panasonic-ELC:ELC18B101L-18B
- added R1, R19, R2, R24, R25, R4, R5, R7: 0.1, standard_passive:RES_1206
- added R17, R22, R27, R32: 0, standard_passive:RES_0603
- added R18, R23, R28, R33: 10k, standard_passive:RES_0603
- added R20, R26, R3, R6: 1M, standard_passive:RES_0603
- added U$1, U$3, U$8, U$9: DRV8825PWP, motor_drivers:DRV8825PWP
- added U2: LM2576HVS-5.0/NOPB-TO263-5, Seeed-OPL-ic:PMIC-LM2576HVS-5.0/NOPB(TO263-5)
- added U5: MCP3204-CI/SL, mcp3204:MCP3204-CI/SL
- added X2, X3, X4, X5, X7: MSTBV4, con-phoenix-508:MSTBV4
- added X6: 87832-14, con-molex:87832-14
Connections:
- removed net +40V1: C47.1, C48.1
- removed net N$34: U3.OUT1@3
- removed net N$35: U3.OUT2@4
- removed net N$36: U3.OUT3@5
- new net +1V2: C29.1, C30.1, C59.1, C60.1, C61.1
- new net +5V: C88.+, L1.1, U2.FEEDBACK
- new net MOT2_DIR: U$1.DIR
- new net MOT2_EN: U$1.ENBL
- new net MOT2_FAULT: R18.1, U$1.FAULT
- new net MOT2_RST: U$1.RESET, U$1.SLEEP
- new net MOT2_STEP: U$1.STEP
- new net MOT2_VREF: C16.1, U$1.AVREF, U$1.BVREF, U3.OUT1@3
- new net MOT3_DIR: U$3.DIR
- new net MOT3_EN: U$3.ENBL
- new net MOT3_FAULT: R23.1, U$3.FAULT
- new net MOT3_RST: U$3.RESET, U$3.SLEEP
- new net MOT3_STEP: U$3.STEP
- new net MOT3_VREF: C26.1, U$3.AVREF, U$3.BVREF, U3.OUT2@4
- new net MOT4_DIR: U$9.DIR
- new net MOT4_EN: U$9.ENBL
- new net MOT4_FAULT: R28.1, U$9.FAULT
- new net MOT4_RST: U$9.RESET, U$9.SLEEP
- new net MOT4_STEP: U$9.STEP
- new net MOT4_VREF: C56.1, U$9.AVREF, U$9.BVREF, U3.OUT3@5
- new net MOT5_DIR: U$8.DIR
- new net MOT5_EN: U$8.ENBL
- new net MOT5_FAULT: R33.1, U$8.FAULT
- new net MOT5_RST: U$8.RESET, U$8.SLEEP
- new net MOT5_STEP: U$8.STEP
- new net MOT5_VREF: C64.1, U$8.AVREF, U$8.BVREF, U3.OUT4@6
- new net N$1: R2.2, U$1.ISENA
- new net N$10: R17.2, U$1.DECAY
- new net N$11: R5.2, U$3.ISENA
- new net N$12: R4.2, U$3.ISENB
- new net N$13: C9.1, U$3.CP1
- new net N$14: C9.2, U$3.CP2
- new net N$15: C10.1, R6.1, U$3.VCP
- new net N$2: R1.2, U$1.ISENB
- new net N$21: U$3.AOUT1, X3-1.1
- new net N$22: U$3.AOUT2, X3-2.1
- new net N$23: U$3.BOUT2, X3-3.1
- new net N$25: U$3.BOUT1, X3-4.1
- new net N$26: R22.2, U$3.DECAY
- new net N$27: R25.2, U$9.ISENA
- new net N$28: R24.2, U$9.ISENB
- new net N$3: C2.1, U$1.CP1
- new net N$33: C31.1, U$9.CP1
- new net N$4: C2.2, U$1.CP2
- new net N$41: C31.2, U$9.CP2
- new net N$42: C50.1, R26.1, U$9.VCP
- new net N$43: U$9.AOUT1, X4-1.1
- new net N$44: U$9.AOUT2, X4-2.1
- new net N$45: U$9.BOUT2, X4-3.1
- new net N$46: U$9.BOUT1, X4-4.1
- new net N$47: R27.2, U$9.DECAY
- new net N$48: R19.2, U$8.ISENA
- new net N$49: R7.2, U$8.ISENB
- new net N$5: C3.1, R3.1, U$1.VCP
- new net N$50: C19.1, U$8.CP1
- new net N$51: C19.2, U$8.CP2
- new net N$52: C20.1, R20.1, U$8.VCP
- new net N$53: U$8.AOUT1, X5-1.1
- new net N$54: U$8.AOUT2, X5-2.1
- new net N$55: U$8.BOUT2, X5-3.1
- new net N$56: U$8.BOUT1, X5-4.1
- new net N$57: R32.2, U$8.DECAY
- new net N$58: U$6.OUT, U1B3.IO_L42N_GCLK24_3
- new net N$6: U$1.AOUT1, X2-1.1
- new net N$7: U$1.AOUT2, X2-2.1
- new net N$8: U$1.BOUT2, X2-3.1
- new net N$9: U$1.BOUT1, X2-4.1
- new net TCK: U1BNA.TCK, X6.6
- new net TDI: U1BNA.TDI, X6.10
- new net TDO: U1BNA.TDO, X6.8
- new net TMS: U1BNA.TMS, X6.4
- net +3V3: now also C11.2, C21.2, C4.2, C51.2, C62.1, C63.1, C67.1, C68.1, C69.1, C70.1, C71.1, C72.1, C73.1, C74.1, C75.1, C76.1, C77.1, C78.1, C79.1, C80.1, C81.1, C82.1, C83.1, C84.1, R17.1, R18.2, R22.1, R23.2, R27.1, R28.2, R32.1, R33.2, U$1.MODE0, U$1.MODE1, U$1.MODE2, U$1.V3P3OUT, U$3.MODE0, U$3.MODE1, U$3.MODE2, U$3.V3P3OUT, U$8.MODE0, U$8.MODE1, U$8.MODE2, U$8.V3P3OUT, U$9.MODE0, U$9.MODE1, U$9.MODE2, U$9.V3P3OUT, U1BVCCAUX.VCCAUX@0, U1BVCCAUX.VCCAUX@1, U1BVCCAUX.VCCAUX@2, U1BVCCAUX.VCCAUX@3, U1BVCCAUX.VCCAUX@4, X6.2
- net +40V: now also C10.2, C12.1, C13.1, C14.+, C15.+, C17.1, C18.1, C20.2, C22.1, C23.1, C24.+, C25.+, C27.1, C28.1, C3.2, C47.1, C48.1, C5.1, C50.2, C52.1, C53.1, C54.+, C55.+, C57.1, C58.1, C6.1, C65.1, C66.1, C7.+, C8.+, C85.+, C86.+, C87.+, R20.2, R26.2, R3.2, R6.2, U$1.VMA, U$1.VMB, U$3.VMA, U$3.VMB, U$8.VMA, U$8.VMB, U$9.VMA, U$9.VMB, U2.VIN, X7-1.1, X7-2.1
- net GND: now also C11.1, C12.2, C13.2, C14.-, C15.-, C16.2, C17.2, C18.2, C21.1, C22.2, C23.2, C24.-, C25.-, C26.2, C27.2, C28.2, C29.2, C30.2, C4.1, C5.2, C51.1, C52.2, C53.2, C54.-, C55.-, C56.2, C57.2, C58.2, C59.2, C6.2, C60.2, C61.2, C62.2, C63.2, C64.2, C65.2, C66.2, C67.2, C68.2, C69.2, C7.-, C70.2, C71.2, C72.2, C73.2, C74.2, C75.2, C76.2, C77.2, C78.2, C79.2, C8.-, C80.2, C81.2, C82.2, C83.2, C84.2, C85.-, C86.-, C87.-, C88.-, D1.A, R1.1, R19.1, R2.1, R24.1, R25.1, R4.1, R5.1, R7.1, U$1.GND_0, U$1.GND_1, U$1.GND_PAD, U$3.GND_0, U$3.GND_1, U$3.GND_PAD, U$8.GND_0, U$8.GND_1, U$8.GND_PAD, U$9.GND_0, U$9.GND_1, U$9.GND_PAD, U1BGND.GND@0, U1BGND.GND@1, U1BGND.GND@10, U1BGND.GND@11, U1BGND.GND@12, U1BGND.GND@2, U1BGND.GND@3, U1BGND.GND@4, U1BGND.GND@5, U1BGND.GND@6, U1BGND.GND@7, U1BGND.GND@8, U1BGND.GND@9, U1BNA.SUSPEND, U2.!ON/OFF, U2.GND, U2.PAD, U5.AGND, U5.DGND, X6.11, X6.13, X6.3, X6.5, X6.7, X6.9, X7-3.1, X7-4.1
- net N$37: now also D1.C, L1.2, U2.OUTPUT; no longer U3.OUT4@6
