File: board/icemot/icemot_v1/icemotv1.sch (EAGLE design)
At the start: 141 parts, among them U1 6SLX9TQG144, U2 LM2576HVS-5.0/NOPB-TO263-5, U3 MAX5723/4/5, U4 TLV4379, U5 MCP3204-CI/SL, X1 MSTBV4, X2 MSTBV4, X3 MSTBV4, X4 MSTBV4, X5 MSTBV4, X6 87832-14, X7 MSTBV4

Commit message: added a 12V rail, Power Mosfet
Parts:
- added C89, C90: (no value), resistor:C-EUC0603
- added C91, C92, C93, C94: (no value), rcl:CPOL-EUE5-10.5
- added D2: MBR360G, diode:SCHOTTKY-DIODEDO201T15
- added L2: 100UH, Panasonic-ELC:ELC18B101L-18B
- added Q1: NTD5805NT4G, infineon_optimos:INFINEON-OPTIMOS-IPD048N96L3G
- added R21: 0, standard_passive:RES_1206
- added R29: 0.01, standard_passive:RES_2512
- added U6: PM8841, pm8841:PM8841
- added U7: LM2576HVS-5.0/NOPB-TO263-5, LM257XHV:PMIC-LM2575HVS-12.0/NOPB(TO263-5)
- added X8: MSTBV4, con-phoenix-508:MSTBV4
- added X9: MST4V, con-phoenix-508:MST4V
Connections:
- new net +12V: C90.1, C94.+, L2.1, U6.VCC, U7.FEEDBACK
- new net FET_1: U6.IN
- new net N$34: Q1.D, X9-1.1
- new net N$35: R21.1, U6.OUT
- new net N$36: Q1.G, R21.2
- new net N$59: X9-2.1, X9-3.1
- new net N$60: Q1.S, R29.2
- new net N$61: D2.C, L2.2, U7.OUTPUT
- net +3V3: now also C89.1, U6.TH
- net +40V: now also C91.+, C92.+, C93.+, U7.VIN, X8-1.1, X8-2.1
- net GND: now also C89.2, C90.2, C91.-, C92.-, C93.-, C94.-, D2.A, R29.1, U6.GND, U7.!ON/OFF, U7.GND, U7.PAD, X8-3.1, X8-4.1, X9-4.1
Other:
- note added: "Bourns: 3W 10mOhm CRA2512-FZ-R010ELF"

Commit message: added ADC and opamp for mosfet
Parts:
- added C100, C101, C102, C99: 1u, standard_passive:CAP_0603
- added C95, C96, C97, C98: (no value), resistor:C-EUC0603
- added Q2, Q3: NTD5805NT4G, infineon_optimos:INFINEON-OPTIMOS-IPD048N96L3G
- added R30, R34: 0, standard_passive:RES_1206
- added R31, R35: 0.01, standard_passive:RES_2512
- added R36, R37, R38, R39: 10, standard_passive:RES_0603
- added R40: 10k, standard_passive:RES_0603
- added U$21: MCP1525T-I/TT, mcp1525:MCP1525T-I/TT
- added U10: MCP3208-CI/SL, mcp3204:MCP3208-CI/SL
- added U8, U9: PM8841, pm8841:PM8841
- added X10, X11: MST4V, con-phoenix-508:MST4V
- U5: value MCP3204-CI/SL -> TLV4379; device mcp3204:MCP3204-CI/SL -> opamp:TLV4379
- U7: value LM2576HVS-5.0/NOPB-TO263-5 -> LM2576HVS-12.0/NOPB-TO263-5
Connections:
- net N$60 renamed CH1_I
- new net ADC_CLK: U10.CLK
- new net ADC_CS: R40.2, U10.*CS/SHDN
- new net ADC_MISO: U10.DOUT
- new net ADC_MOSI: U10.DIN
- new net CH2_I: Q2.S, R31.2
- new net CH3_I: Q3.S, R35.2
- new net FET_2: U8.IN
- new net FET_3: U9.IN
- new net N$62: R30.1, U8.OUT
- new net N$63: Q2.G, R30.2
- new net N$64: Q2.D, X10-1.1
- new net N$65: X10-2.1, X10-3.1
- new net N$67: R34.1, U9.OUT
- new net N$68: Q3.G, R34.2
- new net N$69: Q3.D, X11-1.1
- new net N$70: X11-2.1, X11-3.1
- new net N$72: C100.1, U$21.VOUT, U10.VREF
- new net N$74: R36.1, U10.CH0
- new net N$75: R37.1, U10.CH1
- new net N$76: R38.1, U10.CH2
- new net N$77: R39.1, U10.CH3
- net +12V: now also C96.1, C98.1, U8.VCC, U9.VCC
- net +3V3: now also C101.1, C102.1, C95.1, C97.1, C99.1, R11.2, R12.2, R13.2, R14.2, R40.1, U$21.VIN, U10.VDD, U8.TH, U9.TH; no longer JP1.2, JP2.2, JP3.2, JP4.2
- net GND: now also C100.2, C101.2, C102.2, C95.2, C96.2, C97.2, C98.2, C99.2, JP1.1, JP2.1, JP3.1, JP4.1, R31.1, R35.1, U$21.VSS, U10.AGND, U10.DGND, U8.GND, U9.GND, X10-4.1, X11-4.1; no longer R11.1, R12.1, R13.1, R14.1, U5.AGND, U5.DGND
- net T1_AMP: now also R36.2
- net T1_IN: now also JP1.2, R11.1; no longer JP1.1, R11.2
- net T2_AMP: now also R37.2
- net T2_IN: now also JP2.2, R12.1; no longer JP2.1, R12.2
- net T3_AMP: now also R38.2
- net T3_IN: now also JP3.2, R13.1; no longer JP3.1, R13.2
- net T4_AMP: now also R39.2
- net T4_IN: now also JP4.2, R14.1; no longer JP4.1, R14.2
