File: board/icemot/icemot_v1/icemotv1.brd (EAGLE design)
At the start: 160 x 100 mm, 141 parts, among them U1 6SLX9TQG144, U2 LM2576HVS-5.0/NOPB-TO263-5, U3 MAX5723/4/5, U4 TLV4379, U5 MCP3204-CI/SL, X1 MSTBV4, X2 MSTBV4, X3 MSTBV4, X4 MSTBV4, X5 MSTBV4, X6 87832-14, X7 MSTBV4

Commit message: added a 12V rail, Power Mosfet
Parts:
- added C89, C90: (no value), resistor:C0603
- added C91, C92, C93, C94: (no value), rcl:E5-10,5
- added D2: MBR360G, diode:DO201T15
- added L2: 100UH, Panasonic-ELC:IND_ELC18B
- added Q1: NTD5805NT4G, infineon_optimos:DPAK
- added R21: 0, standard_passive:R1206
- added R29: 0.01, standard_passive:R2512
- added U6: PM8841, pm8841:SOT23-5
- added U7: LM2576HVS-5.0/NOPB-TO263-5, LM257XHV:TO-263-5
- added X8: MSTBV4, con-phoenix-508:MSTBV4
- added X9: MST4V, con-phoenix-508:MSTBV4
- moved X6 47.2 mm to (75.5, 72.0), turned to 180 degrees
Connections:
- new net +12V: C90.1, C94.+, L2.1, U6.1, U7.4
- new net FET_1: U6.3
- new net N$34: Q1.2, X9.1
- new net N$35: R21.1, U6.5
- new net N$36: Q1.1, R21.2
- new net N$59: X9.2, X9.3
- new net N$60: Q1.3, R29.2
- new net N$61: D2.C, L2.2, U7.2
- net +3V3: now also C89.1, U6.4
- net +40V: now also C91.+, C92.+, C93.+, U7.1, X8.1, X8.2
- net GND: now also C89.2, C90.2, C91.-, C92.-, C93.-, C94.-, D2.A, R29.1, U6.2, U7.3, U7.5, U7.PAD, X8.3, X8.4, X9.4

Commit message: added ADC and opamp for mosfet
Parts:
- added C100, C101, C102, C99: 1u, standard_passive:R0603
- added C95, C96, C97, C98: (no value), resistor:C0603
- added Q2, Q3: NTD5805NT4G, infineon_optimos:DPAK
- added R30, R34: 0, standard_passive:R1206
- added R31, R35: 0.01, standard_passive:R2512
- added R36, R37, R38, R39: 10, standard_passive:R0603
- added R40: 10k, standard_passive:R0603
- added U$21: MCP1525T-I/TT, mcp1525:SOT96P237X112-3N
- added U10: MCP3208-CI/SL, mcp3204:SOIC127P600X175-16N
- added U8, U9: PM8841, pm8841:SOT23-5
- added X10, X11: MST4V, con-phoenix-508:MSTBV4
- U5: value MCP3204-CI/SL -> TLV4379; device mcp3204:SOIC127P600X175-14N -> opamp:TSSOP14-0.65-5X4.4MM
- U7: value LM2576HVS-5.0/NOPB-TO263-5 -> LM2576HVS-12.0/NOPB-TO263-5
- moved C91 173.4 mm to (30.0, 73.5)
- moved L2 172.3 mm to (67.0, 41.5)
- moved U5 165.0 mm to (-102.0, -211.0)
- moved D1 145.6 mm to (47.0, 71.0)
- moved C88 142.4 mm to (102.0, 92.5)
- moved L1 91.6 mm to (42.5, 42.0)
Connections:
- net N$60 renamed CH1_I
- removed net VDD: U5.14
- new net ADC_CLK: U10.13
- new net ADC_CS: R40.2, U10.10
- new net ADC_MISO: U10.12
- new net ADC_MOSI: U10.11
- new net CH2_I: Q2.3, R31.2
- new net CH3_I: Q3.3, R35.2
- new net FET_2: U8.3
- new net FET_3: U9.3
- new net N$62: R30.1, U8.5
- new net N$63: Q2.1, R30.2
- new net N$64: Q2.2, X10.1
- new net N$65: X10.2, X10.3
- new net N$67: R34.1, U9.5
- new net N$68: Q3.1, R34.2
- new net N$69: Q3.2, X11.1
- new net N$70: X11.2, X11.3
- new net N$72: C100.1, U$21.2, U10.15
- new net N$74: R36.1, U10.1
- new net N$75: R37.1, U10.2
- new net N$76: R38.1, U10.3
- new net N$77: R39.1, U10.4
- new net V+: U5.4
- new net V-: U5.11
- net +12V: now also C96.1, C98.1, U8.1, U9.1
- net +3V3: now also C101.1, C102.1, C95.1, C97.1, C99.1, R11.2, R12.2, R13.2, R14.2, R40.1, U$21.1, U10.16, U8.4, U9.4; no longer JP1.2, JP2.2, JP3.2, JP4.2
- net GND: now also C100.2, C101.2, C102.2, C95.2, C96.2, C97.2, C98.2, C99.2, JP1.1, JP2.1, JP3.1, JP4.1, R31.1, R35.1, U$21.3, U10.14, U10.9, U8.2, U9.2, X10.4, X11.4; no longer R11.1, R12.1, R13.1, R14.1, U5.12, U5.7
- net T1_AMP: now also R36.2
- net T1_IN: now also JP1.2, R11.1; no longer JP1.1, R11.2
- net T2_AMP: now also R37.2
- net T2_IN: now also JP2.2, R12.1; no longer JP2.1, R12.2
- net T3_AMP: now also R38.2
- net T3_IN: now also JP3.2, R13.1; no longer JP3.1, R13.2
- net T4_AMP: now also R39.2
- net T4_IN: now also JP4.2, R14.1; no longer JP4.1, R14.2
